Commit message: Update my_robot.xacro
Adjusted the dims of the Robot and added some material colors

File: src/my_robot/urdf/my_robot.xacro (robot description, xacro)
@@ -8,9 +8,9 @@
     <child link="chassis" />
   </joint>
-  <link name='chassis'>
+  <link name="chassis">
     <pose>0 0 0.1 0 0 0</pose>
     <inertial>
       <mass value="15.0"/>
-      <origin xyz="0.0 0 0" rpy=" 0 0 0"/>
+      <origin xyz="0.0 0 0" rpy="0 0 0"/>
       <inertia
           ixx="0.1" ixy="0" ixz="0"
@@ -19,164 +19,187 @@
       />
     </inertial>
-    <collision name='collision'>
-      <origin xyz="0 0 0" rpy=" 0 0 0"/>
-      <geometry>
-        <box size=".4 .2 .1"/>
-      </geometry>
-    </collision>
-    <visual name='chassis_visual'>
-      <origin xyz="0 0 0" rpy=" 0 0 0"/>
-      <geometry>
-        <box size=".4 .2 .1"/>
-      </geometry>
-    </visual>
-    <collision name='back_caster_collision'>
-      <origin xyz="-0.15 0 -0.05" rpy=" 0 0 0"/>
-      <geometry>
-        <sphere radius="0.0499"/>
-      </geometry>
-    </collision>
-    <visual name='back_caster_visual'>
-      <origin xyz="-0.15 0 -0.05" rpy=" 0 0 0"/>
-      <geometry>
-        <sphere radius="0.05"/>
-      </geometry>
-    </visual>
-    <collision name='front_caster_collision'>
-      <origin xyz="0.15 0 -0.05" rpy=" 0 0 0"/>
-      <geometry>
-        <sphere radius="0.0499"/>
-      </geometry>
-    </collision>
-    <visual name='front_caster_visual'>
-      <origin xyz="0.15 0 -0.05" rpy=" 0 0 0"/>
-      <geometry>
-        <sphere radius="0.05"/>
-      </geometry>
-    </visual>
-  </link>
-<link name="left_wheel">
-  <inertial>
-    <mass value="5.0"/>
-    <origin xyz="0 0 0" rpy="1.5707 1.5707 0"/>
-    <inertia
-        ixx="0.1" ixy="0" ixz="0"
-        iyy="0.1" iyz="0"
-        izz="0.1"
-    />
-  </inertial>
-  <collision name="left_wheel_collision">
-    <origin xyz="0 0 0" rpy="1.5707 1.5707 0"/>
-    <geometry>
-      <cylinder radius="0.1" length="0.05"/>
-    </geometry>
-  </collision>
-  <visual name="left_wheel_visual">
-    <origin xyz="0 0 0" rpy="1.5707 1.5707 0"/>
-    <geometry>
-      <cylinder radius="0.1" length="0.05"/>
-    </geometry>
-  </visual>
-</link>
-<joint type="continuous" name="left_wheel_hinge">
-  <origin xyz="0 -0.15 0" rpy="0 0 0"/>
-  <child link="left_wheel"/>
-  <parent link="chassis"/>
-  <axis xyz="0 1 0"/> <!-- Rotation around Z-axis -->
-  <limit effort="10000" velocity="1000"/>
-  <dynamics damping="1.0" friction="1.0"/>
-</joint>
-<link name="right_wheel">
-  <inertial>
-    <mass value="5.0"/>
-    <origin xyz="0 0 0" rpy="1.5707 1.5707 0"/>
-    <inertia
-        ixx="0.1" ixy="0" ixz="0"
-        iyy="0.1" iyz="0"
-        izz="0.1"
-    />
-  </inertial>
-  <collision name="right_wheel_collision">
-    <origin xyz="0 0 0" rpy="1.5707 1.5707 0"/>
-    <geometry>
-      <cylinder radius="0.1" length="0.05"/>
-    </geometry>
-  </collision>
-  <visual name="right_wheel_visual">
-    <origin xyz="0 0 0" rpy="1.5707 1.5707 0"/>
-    <geometry>
-      <cylinder radius="0.1" length="0.05"/>
-    </geometry>
-  </visual>
-</link>
-<joint type="continuous" name="right_wheel_hinge">
-  <origin xyz="0 0.15 0" rpy="0 0 0"/>
-  <child link="right_wheel"/>
-  <parent link="chassis"/>
-  <axis xyz="0 1 0"/>
-  <limit effort="10000" velocity="1000"/>
-  <dynamics damping="1.0" friction="1.0"/>
-</joint>
-<!-- Camera Link -->
-<link name="camera">
-  <inertial>
-    <mass value="0.1"/>
-    <origin xyz="0 0 0" rpy="0 0 0"/>
-    <inertia
-        ixx="1e-6" ixy="0" ixz="0"
-        iyy="1e-6" iyz="0"
-        izz="1e-6"
-    />
-  </inertial>
-  <collision>
-    <origin xyz="0 0 0" rpy="0 0 0"/>
-    <geometry>
-      <box size="0.05 0.05 0.05"/>
-    </geometry>
-  </collision>
-  <visual>
-    <origin xyz="0 0 0" rpy="0 0 0"/>
-    <geometry>
-      <box size="0.05 0.05 0.05"/>
-    </geometry>
-  </visual>
-</link>
-<!-- Camera Joint -->
-<joint name="camera_joint" type="fixed">
-  <origin xyz="0.2 0 0" rpy="0 0 0"/>
-  <parent link="chassis"/>
-  <child link="camera"/>
-  <axis xyz="0 1 0"/>
-</joint>
-<!-- Hokuyo LIDAR Link -->
-<link name="hokuyo">
-  <inertial>
-    <mass value="1e-5"/>
-    <origin xyz="0 0 0" rpy="0 0 0"/>
-    <inertia
-        ixx="1e-6" ixy="0" ixz="0"
-        iyy="1e-6" iyz="0"
-        izz="1e-6"
-    />
-  </inertial>
-  <collision>
-    <origin xyz="0 0 0" rpy="0 0 0"/>
-    <geometry>
-      <box size="0.1 0.1 0.1"/>
-    </geometry>
-  </collision>
-  <visual>
-    <origin xyz="0 0 0" rpy="0 0 0"/>
-    <geometry>
-      <mesh filename="package://my_robot/meshes/hokuyo.dae"/>
-    </geometry>
-  </visual>
-</link>
-<!-- Hokuyo LIDAR Joint -->
-<joint name="hokuyo_joint" type="fixed">
-  <origin xyz="0.15 0 0.1" rpy="0 0 0"/>
-  <parent link="chassis"/>
-  <child link="hokuyo"/>
-  <axis xyz="0 1 0"/>
-</joint>
+    <collision name="collision">
+      <origin xyz="0 0 0" rpy="0 0 0"/>
+      <geometry>
+        <box size="0.45 0.3 0.1"/>
+      </geometry>
+    </collision>
+    <visual name="chassis_visual">
+      <origin xyz="0 0 0" rpy="0 0 0"/>
+      <geometry>
+        <box size="0.45 0.3 0.1"/>
+      </geometry>
+      <material name="Blue">
+        <color rgba="0 0 1 1"/>
+      </material>
+    </visual>
+    <collision name="back_caster_collision">
+      <origin xyz="-0.15 0 -0.075" rpy="0 0 0"/>
+      <geometry>
+        <sphere radius="0.0749"/>
+      </geometry>
+    </collision>
+    <visual name="back_caster_visual">
+      <origin xyz="-0.15 0 -0.075" rpy="0 0 0"/>
+      <geometry>
+        <sphere radius="0.075"/>
+      </geometry>
+      <material name="Yellow">
+        <color rgba="1 1 0 1"/>
+      </material>
+    </visual>
+    <collision name="front_caster_collision">
+      <origin xyz="0.15 0 -0.075" rpy="0 0 0"/>
+      <geometry>
+        <sphere radius="0.0749"/>
+      </geometry>
+    </collision>
+    <visual name="front_caster_visual">
+      <origin xyz="0.15 0 -0.075" rpy="0 0 0"/>
+      <geometry>
+        <sphere radius="0.075"/>
+      </geometry>
+      <material name="Yellow">
+        <color rgba="1 1 0 1"/>
+      </material>
+    </visual>
+  </link>
+  <link name="left_wheel">
+    <inertial>
+      <mass value="5.0"/>
+      <origin xyz="0 0 0" rpy="0 0 0"/>
+      <inertia
+          ixx="0.1" ixy="0" ixz="0"
+          iyy="0.1" iyz="0"
+          izz="0.1"
+      />
+    </inertial>
+    <collision name="left_wheel_collision">
+      <origin xyz="0 0 0" rpy="0 1.5707 1.5707"/>
+      <geometry>
+        <cylinder radius="0.15" length="0.05"/>
+      </geometry>
+    </collision>
+    <visual name="left_wheel_visual">
+      <origin xyz="0 0 0" rpy="0 1.5707 1.5707"/>
+      <geometry>
+        <cylinder radius="0.15" length="0.05"/>
+      </geometry>
+      <material name="Green">
+        <color rgba="0 1 0 1"/>
+      </material>
+    </visual>
+  </link>
+  <!-- LEFT WHEEL JOINT -->
+  <joint type="continuous" name="left_wheel_hinge">
+    <origin xyz="0 0.2 0" rpy="0 0 0"/>
+    <child link="left_wheel"/>
+    <parent link="chassis"/>
+    <axis xyz="0 1 0"/>
+    <limit effort="10000" velocity="1000"/>
+    <dynamics damping="1.0" friction="1.0"/>
+  </joint>
+  <!-- RIGHT WHEEL LINK -->
+  <link name="right_wheel">
+    <inertial>
+      <mass value="5.0"/>
+      <origin xyz="0 0 0" rpy="0 0 0"/>
+      <inertia
+          ixx="0.1" ixy="0" ixz="0"
+          iyy="0.1" iyz="0"
+          izz="0.1"
+      />
+    </inertial>
+    <collision name="right_wheel_collision">
+      <origin xyz="0 0 0" rpy="0 1.5708 1.5708"/>
+      <geometry>
+        <!-- Wheel radius remains 0.15 -->
+        <cylinder radius="0.15" length="0.05"/>
+      </geometry>
+    </collision>
+    <visual name="right_wheel_visual">
+      <origin xyz="0 0 0" rpy="0 1.5707 1.5707"/>
+      <geometry>
+        <cylinder radius="0.15" length="0.05"/>
+      </geometry>
+      <!-- Green wheels -->
+      <material name="Green">
+        <color rgba="0 1 0 1"/>
+      </material>
+    </visual>
+  </link>
+  <!-- RIGHT WHEEL JOINT -->
+  <joint type="continuous" name="right_wheel_hinge">
+    <origin xyz="0 -0.2 0" rpy="0 0 0"/>
+    <child link="right_wheel"/>
+    <parent link="chassis"/>
+    <axis xyz="0 1 0"/>
+    <limit effort="10000" velocity="1000"/>
+    <dynamics damping="1.0" friction="1.0"/>
+  </joint>
+  <!-- CAMERA LINK -->
+  <link name="camera">
+    <inertial>
+      <mass value="0.1"/>
+      <origin xyz="0 0 0" rpy="0 0 0"/>
+      <inertia
+          ixx="1e-6" ixy="0" ixz="0"
+          iyy="1e-6" iyz="0"
+          izz="1e-6"
+      />
+    </inertial>
+    <collision>
+      <origin xyz="0 0 0" rpy="0 0 0"/>
+      <geometry>
+        <box size="0.05 0.05 0.05"/>
+      </geometry>
+    </collision>
+    <visual>
+      <origin xyz="0 0 0" rpy="0 0 0"/>
+      <geometry>
+        <box size="0.05 0.05 0.05"/>
+      </geometry>
+      <material name="Red">
+        <color rgba="1 0 0 1"/>
+      </material>
+    </visual>
+  </link>
+  <!-- CAMERA JOINT -->
+  <joint name="camera_joint" type="fixed">
+    <origin xyz="0.25 0 0" rpy="0 0 0"/>
+    <parent link="chassis"/>
+    <child link="camera"/>
+    <axis xyz="0 1 0"/>
+  </joint>
+  <!-- HOKUYO LIDAR LINK -->
+  <link name="hokuyo">
+    <inertial>
+      <mass value="1e-5"/>
+      <origin xyz="0 0 0" rpy="0 0 0"/>
+      <inertia
+          ixx="1e-6" ixy="0" ixz="0"
+          iyy="1e-6" iyz="0"
+          izz="1e-6"
+      />
+    </inertial>
+    <collision>
+      <origin xyz="0 0 0" rpy="0 0 0"/>
+      <geometry>
+        <box size="0.1 0.1 0.1"/>
+      </geometry>
+    </collision>
+    <visual>
+      <origin xyz="0 0 0" rpy="0 0 0"/>
+      <geometry>
+        <mesh filename="package://my_robot/meshes/hokuyo.dae"/>
+      </geometry>
+    </visual>
+  </link>
+  <!-- HOKUYO LIDAR JOINT -->
+  <joint name="hokuyo_joint" type="fixed">
+    <origin xyz="0.2 0 0.1" rpy="0 0 0"/>
+    <parent link="chassis"/>
+    <child link="hokuyo"/>
+    <axis xyz="0 1 0"/>
+  </joint>
 </robot>

Commit message: Update my_robot.xacro
Added gazebo Specific colors to the robot URDF.

File: src/my_robot/urdf/my_robot.xacro (robot description, xacro)
@@ -30,6 +30,6 @@
         <box size="0.45 0.3 0.1"/>
       </geometry>
-      <material name="Blue">
-        <color rgba="0 0 1 1"/>
+      <material name="bright_red">
+        <color rgba="1 0 0 1"/>
       </material>
     </visual>
@@ -45,5 +45,5 @@
         <sphere radius="0.075"/>
       </geometry>
-      <material name="Yellow">
+      <material name="">
         <color rgba="1 1 0 1"/>
       </material>
@@ -60,5 +60,5 @@
         <sphere radius="0.075"/>
       </geometry>
-      <material name="Yellow">
+      <material name="">
         <color rgba="1 1 0 1"/>
       </material>
@@ -203,3 +203,19 @@
     <axis xyz="0 1 0"/>
   </joint>
+  <!-- Gazebo color Chasis -->
+  <gazebo reference="chassis">
+    <material>Gazebo/Blue</material>
+  </gazebo>
+  <!-- GAZEBOleft wheel -->
+    <gazebo reference="left_wheel">
+      <material>Gazebo/Green</material>
+    </gazebo>
+  <!-- GAZEBO right wheel -->
+    <gazebo reference="right_wheel">
+      <material>Gazebo/Green</material>
+    </gazebo>
+  <!-- GAZEBO color camera -->
+    <gazebo reference="camera">
+      <material>Gazebo/Red</material>
+    </gazebo>
 </robot>

Commit message: Added ball_chaser and my_robot packages

File: src/my_robot/urdf/my_robot.xacro (robot description, xacro)
@@ -8,9 +8,9 @@
     <child link="chassis" />
   </joint>
-  <link name='chassis'>
+  <link name="chassis">
     <pose>0 0 0.1 0 0 0</pose>
     <inertial>
       <mass value="15.0"/>
-      <origin xyz="0.0 0 0" rpy=" 0 0 0"/>
+      <origin xyz="0.0 0 0" rpy="0 0 0"/>
       <inertia
           ixx="0.1" ixy="0" ixz="0"
@@ -19,164 +19,203 @@
       />
     </inertial>
-    <collision name='collision'>
-      <origin xyz="0 0 0" rpy=" 0 0 0"/>
-      <geometry>
-        <box size=".4 .2 .1"/>
-      </geometry>
-    </collision>
-    <visual name='chassis_visual'>
-      <origin xyz="0 0 0" rpy=" 0 0 0"/>
-      <geometry>
-        <box size=".4 .2 .1"/>
-      </geometry>
-    </visual>
-    <collision name='back_caster_collision'>
-      <origin xyz="-0.15 0 -0.05" rpy=" 0 0 0"/>
-      <geometry>
-        <sphere radius="0.0499"/>
-      </geometry>
-    </collision>
-    <visual name='back_caster_visual'>
-      <origin xyz="-0.15 0 -0.05" rpy=" 0 0 0"/>
-      <geometry>
-        <sphere radius="0.05"/>
-      </geometry>
-    </visual>
-    <collision name='front_caster_collision'>
-      <origin xyz="0.15 0 -0.05" rpy=" 0 0 0"/>
-      <geometry>
-        <sphere radius="0.0499"/>
-      </geometry>
-    </collision>
-    <visual name='front_caster_visual'>
-      <origin xyz="0.15 0 -0.05" rpy=" 0 0 0"/>
-      <geometry>
-        <sphere radius="0.05"/>
-      </geometry>
-    </visual>
-  </link>
-<link name="left_wheel">
-  <inertial>
-    <mass value="5.0"/>
-    <origin xyz="0 0 0" rpy="1.5707 1.5707 0"/>
-    <inertia
-        ixx="0.1" ixy="0" ixz="0"
-        iyy="0.1" iyz="0"
-        izz="0.1"
-    />
-  </inertial>
-  <collision name="left_wheel_collision">
-    <origin xyz="0 0 0" rpy="1.5707 1.5707 0"/>
-    <geometry>
-      <cylinder radius="0.1" length="0.05"/>
-    </geometry>
-  </collision>
-  <visual name="left_wheel_visual">
-    <origin xyz="0 0 0" rpy="1.5707 1.5707 0"/>
-    <geometry>
-      <cylinder radius="0.1" length="0.05"/>
-    </geometry>
-  </visual>
-</link>
-<joint type="continuous" name="left_wheel_hinge">
-  <origin xyz="0 -0.15 0" rpy="0 0 0"/>
-  <child link="left_wheel"/>
-  <parent link="chassis"/>
-  <axis xyz="0 1 0"/> <!-- Rotation around Z-axis -->
-  <limit effort="10000" velocity="1000"/>
-  <dynamics damping="1.0" friction="1.0"/>
-</joint>
-<link name="right_wheel">
-  <inertial>
-    <mass value="5.0"/>
-    <origin xyz="0 0 0" rpy="1.5707 1.5707 0"/>
-    <inertia
-        ixx="0.1" ixy="0" ixz="0"
-        iyy="0.1" iyz="0"
-        izz="0.1"
-    />
-  </inertial>
-  <collision name="right_wheel_collision">
-    <origin xyz="0 0 0" rpy="1.5707 1.5707 0"/>
-    <geometry>
-      <cylinder radius="0.1" length="0.05"/>
-    </geometry>
-  </collision>
-  <visual name="right_wheel_visual">
-    <origin xyz="0 0 0" rpy="1.5707 1.5707 0"/>
-    <geometry>
-      <cylinder radius="0.1" length="0.05"/>
-    </geometry>
-  </visual>
-</link>
-<joint type="continuous" name="right_wheel_hinge">
-  <origin xyz="0 0.15 0" rpy="0 0 0"/>
-  <child link="right_wheel"/>
-  <parent link="chassis"/>
-  <axis xyz="0 1 0"/>
-  <limit effort="10000" velocity="1000"/>
-  <dynamics damping="1.0" friction="1.0"/>
-</joint>
-<!-- Camera Link -->
-<link name="camera">
-  <inertial>
-    <mass value="0.1"/>
-    <origin xyz="0 0 0" rpy="0 0 0"/>
-    <inertia
-        ixx="1e-6" ixy="0" ixz="0"
-        iyy="1e-6" iyz="0"
-        izz="1e-6"
-    />
-  </inertial>
-  <collision>
-    <origin xyz="0 0 0" rpy="0 0 0"/>
-    <geometry>
-      <box size="0.05 0.05 0.05"/>
-    </geometry>
-  </collision>
-  <visual>
-    <origin xyz="0 0 0" rpy="0 0 0"/>
-    <geometry>
-      <box size="0.05 0.05 0.05"/>
-    </geometry>
-  </visual>
-</link>
-<!-- Camera Joint -->
-<joint name="camera_joint" type="fixed">
-  <origin xyz="0.2 0 0" rpy="0 0 0"/>
-  <parent link="chassis"/>
-  <child link="camera"/>
-  <axis xyz="0 1 0"/>
-</joint>
-<!-- Hokuyo LIDAR Link -->
-<link name="hokuyo">
-  <inertial>
-    <mass value="1e-5"/>
-    <origin xyz="0 0 0" rpy="0 0 0"/>
-    <inertia
-        ixx="1e-6" ixy="0" ixz="0"
-        iyy="1e-6" iyz="0"
-        izz="1e-6"
-    />
-  </inertial>
-  <collision>
-    <origin xyz="0 0 0" rpy="0 0 0"/>
-    <geometry>
-      <box size="0.1 0.1 0.1"/>
-    </geometry>
-  </collision>
-  <visual>
-    <origin xyz="0 0 0" rpy="0 0 0"/>
-    <geometry>
-      <mesh filename="package://my_robot/meshes/hokuyo.dae"/>
-    </geometry>
-  </visual>
-</link>
-<!-- Hokuyo LIDAR Joint -->
-<joint name="hokuyo_joint" type="fixed">
-  <origin xyz="0.15 0 0.1" rpy="0 0 0"/>
-  <parent link="chassis"/>
-  <child link="hokuyo"/>
-  <axis xyz="0 1 0"/>
-</joint>
+    <collision name="collision">
+      <origin xyz="0 0 0" rpy="0 0 0"/>
+      <geometry>
+        <box size="0.45 0.3 0.1"/>
+      </geometry>
+    </collision>
+    <visual name="chassis_visual">
+      <origin xyz="0 0 0" rpy="0 0 0"/>
+      <geometry>
+        <box size="0.45 0.3 0.1"/>
+      </geometry>
+      <material name="bright_red">
+        <color rgba="1 0 0 1"/>
+      </material>
+    </visual>
+    <collision name="back_caster_collision">
+      <origin xyz="-0.15 0 -0.075" rpy="0 0 0"/>
+      <geometry>
+        <sphere radius="0.0749"/>
+      </geometry>
+    </collision>
+    <visual name="back_caster_visual">
+      <origin xyz="-0.15 0 -0.075" rpy="0 0 0"/>
+      <geometry>
+        <sphere radius="0.075"/>
+      </geometry>
+      <material name="">
+        <color rgba="1 1 0 1"/>
+      </material>
+    </visual>
+    <collision name="front_caster_collision">
+      <origin xyz="0.15 0 -0.075" rpy="0 0 0"/>
+      <geometry>
+        <sphere radius="0.0749"/>
+      </geometry>
+    </collision>
+    <visual name="front_caster_visual">
+      <origin xyz="0.15 0 -0.075" rpy="0 0 0"/>
+      <geometry>
+        <sphere radius="0.075"/>
+      </geometry>
+      <material name="">
+        <color rgba="1 1 0 1"/>
+      </material>
+    </visual>
+  </link>
+  <link name="left_wheel">
+    <inertial>
+      <mass value="5.0"/>
+      <origin xyz="0 0 0" rpy="0 0 0"/>
+      <inertia
+          ixx="0.1" ixy="0" ixz="0"
+          iyy="0.1" iyz="0"
+          izz="0.1"
+      />
+    </inertial>
+    <collision name="left_wheel_collision">
+      <origin xyz="0 0 0" rpy="0 1.5707 1.5707"/>
+      <geometry>
+        <cylinder radius="0.15" length="0.05"/>
+      </geometry>
+    </collision>
+    <visual name="left_wheel_visual">
+      <origin xyz="0 0 0" rpy="0 1.5707 1.5707"/>
+      <geometry>
+        <cylinder radius="0.15" length="0.05"/>
+      </geometry>
+      <material name="Green">
+        <color rgba="0 1 0 1"/>
+      </material>
+    </visual>
+  </link>
+  <!-- LEFT WHEEL JOINT -->
+  <joint type="continuous" name="left_wheel_hinge">
+    <origin xyz="0 0.2 0" rpy="0 0 0"/>
+    <child link="left_wheel"/>
+    <parent link="chassis"/>
+    <axis xyz="0 1 0"/>
+    <limit effort="10000" velocity="1000"/>
+    <dynamics damping="1.0" friction="1.0"/>
+  </joint>
+  <!-- RIGHT WHEEL LINK -->
+  <link name="right_wheel">
+    <inertial>
+      <mass value="5.0"/>
+      <origin xyz="0 0 0" rpy="0 0 0"/>
+      <inertia
+          ixx="0.1" ixy="0" ixz="0"
+          iyy="0.1" iyz="0"
+          izz="0.1"
+      />
+    </inertial>
+    <collision name="right_wheel_collision">
+      <origin xyz="0 0 0" rpy="0 1.5708 1.5708"/>
+      <geometry>
+        <!-- Wheel radius remains 0.15 -->
+        <cylinder radius="0.15" length="0.05"/>
+      </geometry>
+    </collision>
+    <visual name="right_wheel_visual">
+      <origin xyz="0 0 0" rpy="0 1.5707 1.5707"/>
+      <geometry>
+        <cylinder radius="0.15" length="0.05"/>
+      </geometry>
+      <!-- Green wheels -->
+      <material name="Green">
+        <color rgba="0 1 0 1"/>
+      </material>
+    </visual>
+  </link>
+  <!-- RIGHT WHEEL JOINT -->
+  <joint type="continuous" name="right_wheel_hinge">
+    <origin xyz="0 -0.2 0" rpy="0 0 0"/>
+    <child link="right_wheel"/>
+    <parent link="chassis"/>
+    <axis xyz="0 1 0"/>
+    <limit effort="10000" velocity="1000"/>
+    <dynamics damping="1.0" friction="1.0"/>
+  </joint>
+  <!-- CAMERA LINK -->
+  <link name="camera">
+    <inertial>
+      <mass value="0.1"/>
+      <origin xyz="0 0 0" rpy="0 0 0"/>
+      <inertia
+          ixx="1e-6" ixy="0" ixz="0"
+          iyy="1e-6" iyz="0"
+          izz="1e-6"
+      />
+    </inertial>
+    <collision>
+      <origin xyz="0 0 0" rpy="0 0 0"/>
+      <geometry>
+        <box size="0.05 0.05 0.05"/>
+      </geometry>
+    </collision>
+    <visual>
+      <origin xyz="0 0 0" rpy="0 0 0"/>
+      <geometry>
+        <box size="0.05 0.05 0.05"/>
+      </geometry>
+      <material name="Red">
+        <color rgba="1 0 0 1"/>
+      </material>
+    </visual>
+  </link>
+  <!-- CAMERA JOINT -->
+  <joint name="camera_joint" type="fixed">
+    <origin xyz="0.25 0 0" rpy="0 0 0"/>
+    <parent link="chassis"/>
+    <child link="camera"/>
+    <axis xyz="0 1 0"/>
+  </joint>
+  <!-- HOKUYO LIDAR LINK -->
+  <link name="hokuyo">
+    <inertial>
+      <mass value="1e-5"/>
+      <origin xyz="0 0 0" rpy="0 0 0"/>
+      <inertia
+          ixx="1e-6" ixy="0" ixz="0"
+          iyy="1e-6" iyz="0"
+          izz="1e-6"
+      />
+    </inertial>
+    <collision>
+      <origin xyz="0 0 0" rpy="0 0 0"/>
+      <geometry>
+        <box size="0.1 0.1 0.1"/>
+      </geometry>
+    </collision>
+    <visual>
+      <origin xyz="0 0 0" rpy="0 0 0"/>
+      <geometry>
+        <mesh filename="package://my_robot/meshes/hokuyo.dae"/>
+      </geometry>
+    </visual>
+  </link>
+  <!-- HOKUYO LIDAR JOINT -->
+  <joint name="hokuyo_joint" type="fixed">
+    <origin xyz="0.2 0 0.1" rpy="0 0 0"/>
+    <parent link="chassis"/>
+    <child link="hokuyo"/>
+    <axis xyz="0 1 0"/>
+  </joint>
+  <!-- Gazebo color Chasis -->
+  <gazebo reference="chassis">
+    <material>Gazebo/Blue</material>
+  </gazebo>
+  <!-- GAZEBOleft wheel -->
+    <gazebo reference="left_wheel">
+      <material>Gazebo/Green</material>
+    </gazebo>
+  <!-- GAZEBO right wheel -->
+    <gazebo reference="right_wheel">
+      <material>Gazebo/Green</material>
+    </gazebo>
+  <!-- GAZEBO color camera -->
+    <gazebo reference="camera">
+      <material>Gazebo/Red</material>
+    </gazebo>
 </robot>

Commit message: added loclization and mapping launch files and edited the urdf to include depth cam

File: src/my_robot/urdf/my_robot.xacro (robot description, xacro)
@@ -172,4 +172,13 @@
     <axis xyz="0 1 0"/>
   </joint>
+  <!-- CAMERA OPTICAL JOINT-->
+  <joint name="camera_optical_joint" type="fixed">
+    <origin xyz="0 0 0" rpy="-1.5707 0 -1.5707"/>
+    <parent link="camera"/>
+    <child link="camera_link_optical"/>
+  </joint>
+  <!-- CAMERA OPTICAL LINK -->
+  <link name="camera_link_optical">
+  </link>
   <!-- HOKUYO LIDAR LINK -->
   <link name="hokuyo">
